File: new-keyboard-pcb/matrix.kicad_sch (KiCad schematic)
At the start: 198 parts, among them SW1 ESC, SW10 F9, SW11 F10, SW12 F11, SW13 F12, SW14 PWR, SW15 NUMLCK, SW16 DIV, SW17 MULT, SW18 SUB, SW19 /, SW2 F1, SW20 1, SW21 2, SW22 3, SW23 4, SW24 5, SW25 6, SW26 7, SW27 8, SW28 9, SW29 0, SW3 F2, SW30 -, SW31 =, SW32 DEL, SW33 #7, SW34 #8, SW35 #9, SW36 TAB, SW37 Q, SW38 W, SW39 E, SW4 F3, SW40 R, SW41 T, SW42 Y, SW43 U, SW44 I, SW45 O, SW46 P, SW47 ^, SW48 Ç, SW49 ENTER, SW5 F4, SW50 #4, SW51 #5, SW52 #6, SW53 ADD, SW54 CAPSLCK, SW55 A, SW56 S, SW57 D, SW58 F, SW59 G, SW6 F5, SW60 H, SW61 J, SW62 K, SW63 L, SW64 ;, SW65 È, SW66 À, SW67 ENTER, SW68 #1, SW69 #2, SW7 F6, SW70 #3, SW71 #ENTER, SW72 LSHFT, SW73 Ù, SW74 Z, SW75 X, SW76 C, SW77 V, SW78 B, SW79 N, SW8 F7, SW80 M, SW81 ,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

Commit message: midway correcting hotswap sockets
Connections:
- net ROW0B: no longer D15.1 (K), D16.1 (K), D17.1 (K), D18.1 (K)
- net ROW1B: no longer D33.1 (K), D34.1 (K), D35.1 (K)
- net ROW2B: no longer D50.1 (K), D51.1 (K), D52.1 (K), D53.1 (K)
- net ROW3B: no longer D68.1 (K), D69.1 (K), D70.1 (K), D71.1 (K)
- net ROW4B: no longer D85.1 (K), D86.1 (K)
- net ROW5A: no longer D91.1 (K)
- net ROW5B: now also D91.1 (K); no longer D96.1 (K), D97.1 (K), D98.1 (K), D99.1 (K)
- new net ROW0C: D15.1 (K), D16.1 (K), D17.1 (K), D18.1 (K)
- new net ROW1C: D33.1 (K), D34.1 (K), D35.1 (K)
- new net ROW2C: D50.1 (K), D51.1 (K), D52.1 (K), D53.1 (K)
- new net ROW3C: D68.1 (K), D69.1 (K), D70.1 (K), D71.1 (K)
- new net ROW4C: D85.1 (K), D86.1 (K)
- new net ROW5C: D96.1 (K), D97.1 (K), D98.1 (K), D99.1 (K)
