File: new-keyboard-pcb/new-keyboard-pcb.kicad_pcb (KiCad board)
At the start: 2 copper layers, 74.1 x 38.6 mm, 24 parts, among them SW1 SW_Push, U1 ATmega32U4-A, Y1 16MHz

Commit message: return to masterzen
Parts:
- removed C1, C2: 22pF, Capacitor_SMD:C_0805_2012Metric_Pad1.18x1.45mm_HandSolder
- removed C3: 1µF, Capacitor_SMD:C_0805_2012Metric_Pad1.18x1.45mm_HandSolder
- removed C4, C5, C6, C7: 0.1µF, Capacitor_SMD:C_0805_2012Metric_Pad1.18x1.45mm_HandSolder
- removed CH1, CH2, CH3, CH4: choc_v1_SW_HS, Kailh_PG1353_Hotswap:Kailh-PG1353-Hotswap-1U
- removed D1, D2, D3, D4: D_Small, Diode_SMD:D_SOD-123
- removed F1: 500mA, Fuse:Fuse_1206_3216Metric_Pad1.42x1.75mm_HandSolder
- removed R1, R4: 10k, Resistor_SMD:R_0805_2012Metric_Pad1.20x1.40mm_HandSolder
- removed R2, R3: 22, Resistor_SMD:R_0805_2012Metric_Pad1.20x1.40mm_HandSolder
- removed SW1: SW_Push, random-keyboard-parts.pretty-master:SKQG-1155865
- removed U1: ATmega32U4-A, Package_QFP:TQFP-44_10x10mm_P0.8mm
- removed USB1: Molex-0548190589, random-keyboard-parts.pretty-master:Molex-0548190589
- removed Y1: 16MHz, Crystal:Crystal_SMD_3225-4Pin_3.2x2.5mm_HandSoldering
Routing:
- net GND: track 123.5 -> 0.00 mm
- net +5V: track 82.5 -> 0.00 mm, vias 5 -> 0
- net ROW0: track 54.7 -> 0.00 mm
- net COL1: track 53.1 -> 0.00 mm, vias 1 -> 0
- net ROW1: track 48.5 -> 0.00 mm
- net COL0: track 29.5 -> 0.00 mm, vias 1 -> 0
- net Net-(U1-~{RESET}): track 24.3 -> 0.00 mm, vias 2 -> 0
- net Net-(U1-D-): track 22.8 -> 0.00 mm
- net Net-(U1-D+): track 22.1 -> 0.00 mm
- net VCC: track 12.4 -> 0.00 mm
- net Net-(U1-XTAL2): track 11.5 -> 0.00 mm
- net Net-(U1-XTAL1): track 9.35 -> 0.00 mm
- net Net-(D1-A): track 5.87 -> 0.00 mm, vias 1 -> 0
- net Net-(D4-A): track 5.73 -> 0.00 mm, vias 1 -> 0
- net Net-(D3-A): track 5.73 -> 0.00 mm, vias 1 -> 0
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Other:
- board outline removed

Commit message: main keyboard switch placed
Parts:
- added C1: 22pF, Capacitor_SMD:C_0805_2012Metric_Pad1.18x1.45mm_HandSolder, F.Cu at (-134.1, 166.2)
- added C2: 22pF, Capacitor_SMD:C_0805_2012Metric_Pad1.18x1.45mm_HandSolder, F.Cu at (-134.1, 169.2)
- added C3: 1µF, Capacitor_SMD:C_0805_2012Metric_Pad1.18x1.45mm_HandSolder, F.Cu at (-134.1, 172.3)
- added C4: 0.1µF, Capacitor_SMD:C_0805_2012Metric_Pad1.18x1.45mm_HandSolder, F.Cu at (-134.1, 175.3)
- added C5: 0.1µF, Capacitor_SMD:C_0805_2012Metric_Pad1.18x1.45mm_HandSolder, F.Cu at (-134.1, 178.3)
- added C6: 0.1µF, Capacitor_SMD:C_0805_2012Metric_Pad1.18x1.45mm_HandSolder, F.Cu at (-134.1, 181.3)
- added C7: 1µF, Capacitor_SMD:C_0805_2012Metric_Pad1.18x1.45mm_HandSolder, F.Cu at (-134.1, 184.3)
- added C8: 1µF, Capacitor_SMD:C_0805_2012Metric_Pad1.18x1.45mm_HandSolder, F.Cu at (-134.1, 187.3)
- added C9: 1µF, Capacitor_SMD:C_0805_2012Metric_Pad1.18x1.45mm_HandSolder, F.Cu at (-134.1, 190.3)
- added D1: D_Small, Diode_SMD:D_0805_2012Metric_Pad1.15x1.40mm_HandSolder, F.Cu at (-62.5, 159.1)
- added D10: D_Small, Diode_SMD:D_0805_2012Metric_Pad1.15x1.40mm_HandSolder, F.Cu at (-62.5, 186.4)
- added D11: D_Small, Diode_SMD:D_0805_2012Metric_Pad1.15x1.40mm_HandSolder, F.Cu at (-62.5, 189.5)
- added D12: D_Small, Diode_SMD:D_0805_2012Metric_Pad1.15x1.40mm_HandSolder, F.Cu at (-62.5, 192.5)
- added D13: D_Small, Diode_SMD:D_0805_2012Metric_Pad1.15x1.40mm_HandSolder, F.Cu at (-62.5, 195.5)
- added D14: D_Small, Diode_SMD:D_0805_2012Metric_Pad1.15x1.40mm_HandSolder, F.Cu at (-57.7, 159.1)
- added D15: D_Small, Diode_SMD:D_0805_2012Metric_Pad1.15x1.40mm_HandSolder, F.Cu at (-57.7, 162.1)
- added D16: D_Small, Diode_SMD:D_0805_2012Metric_Pad1.15x1.40mm_HandSolder, F.Cu at (-57.7, 165.1)
- added D17: D_Small, Diode_SMD:D_0805_2012Metric_Pad1.15x1.40mm_HandSolder, F.Cu at (-57.7, 168.2)
- added D18: D_Small, Diode_SMD:D_0805_2012Metric_Pad1.15x1.40mm_HandSolder, F.Cu at (-57.7, 171.2)
- added D19: D_Small, Diode_SMD:D_0805_2012Metric_Pad1.15x1.40mm_HandSolder, F.Cu at (-57.7, 174.3)
- added D2: D_Small, Diode_SMD:D_0805_2012Metric_Pad1.15x1.40mm_HandSolder, F.Cu at (-62.5, 162.1)
- added D20: D_Small, Diode_SMD:D_0805_2012Metric_Pad1.15x1.40mm_HandSolder, F.Cu at (-57.7, 177.3)
- added D21: D_Small, Diode_SMD:D_0805_2012Metric_Pad1.15x1.40mm_HandSolder, F.Cu at (-57.7, 180.3)
- added D22: D_Small, Diode_SMD:D_0805_2012Metric_Pad1.15x1.40mm_HandSolder, F.Cu at (-57.7, 183.4)
- added D23: D_Small, Diode_SMD:D_0805_2012Metric_Pad1.15x1.40mm_HandSolder, F.Cu at (-57.7, 186.4)
- added D24: D_Small, Diode_SMD:D_0805_2012Metric_Pad1.15x1.40mm_HandSolder, F.Cu at (-57.7, 189.5)
- added D25: D_Small, Diode_SMD:D_0805_2012Metric_Pad1.15x1.40mm_HandSolder, F.Cu at (-57.7, 192.5)
- added D26: D_Small, Diode_SMD:D_0805_2012Metric_Pad1.15x1.40mm_HandSolder, F.Cu at (-57.7, 195.5)
- added D27: D_Small, Diode_SMD:D_0805_2012Metric_Pad1.15x1.40mm_HandSolder, F.Cu at (-52.9, 159.1)
- added D28: D_Small, Diode_SMD:D_0805_2012Metric_Pad1.15x1.40mm_HandSolder, F.Cu at (-52.9, 162.1)
- added D29: D_Small, Diode_SMD:D_0805_2012Metric_Pad1.15x1.40mm_HandSolder, F.Cu at (-52.9, 165.1)
- added D3: D_Small, Diode_SMD:D_0805_2012Metric_Pad1.15x1.40mm_HandSolder, F.Cu at (-62.5, 165.1)
- added D30: D_Small, Diode_SMD:D_0805_2012Metric_Pad1.15x1.40mm_HandSolder, F.Cu at (-52.9, 168.2)
- added D31: D_Small, Diode_SMD:D_0805_2012Metric_Pad1.15x1.40mm_HandSolder, F.Cu at (-52.9, 171.2)
- added D32: D_Small, Diode_SMD:D_0805_2012Metric_Pad1.15x1.40mm_HandSolder, F.Cu at (-52.9, 174.3)
- added D33: D_Small, Diode_SMD:D_0805_2012Metric_Pad1.15x1.40mm_HandSolder, F.Cu at (-52.9, 177.3)
- added D34: D_Small, Diode_SMD:D_0805_2012Metric_Pad1.15x1.40mm_HandSolder, F.Cu at (-52.9, 180.3)
- added D35: D_Small, Diode_SMD:D_0805_2012Metric_Pad1.15x1.40mm_HandSolder, F.Cu at (-52.9, 183.4)
- added D36: D_Small, Diode_SMD:D_0805_2012Metric_Pad1.15x1.40mm_HandSolder, F.Cu at (-52.9, 186.4)
- added D37: D_Small, Diode_SMD:D_0805_2012Metric_Pad1.15x1.40mm_HandSolder, F.Cu at (-52.9, 189.5)
- added D38: D_Small, Diode_SMD:D_0805_2012Metric_Pad1.15x1.40mm_HandSolder, F.Cu at (-52.9, 192.5)
- added D39: D_Small, Diode_SMD:D_0805_2012Metric_Pad1.15x1.40mm_HandSolder, F.Cu at (-52.9, 195.5)
- added D4: D_Small, Diode_SMD:D_0805_2012Metric_Pad1.15x1.40mm_HandSolder, F.Cu at (-62.5, 168.2)
- added D40: D_Small, Diode_SMD:D_0805_2012Metric_Pad1.15x1.40mm_HandSolder, F.Cu at (-48.1, 159.1)
- added D41: D_Small, Diode_SMD:D_0805_2012Metric_Pad1.15x1.40mm_HandSolder, F.Cu at (-48.1, 162.1)
- added D42: D_Small, Diode_SMD:D_0805_2012Metric_Pad1.15x1.40mm_HandSolder, F.Cu at (-48.1, 165.1)
- added D43: D_Small, Diode_SMD:D_0805_2012Metric_Pad1.15x1.40mm_HandSolder, F.Cu at (-48.1, 168.2)
- added D44: D_Small, Diode_SMD:D_0805_2012Metric_Pad1.15x1.40mm_HandSolder, F.Cu at (-48.1, 171.2)
- added D45: D_Small, Diode_SMD:D_0805_2012Metric_Pad1.15x1.40mm_HandSolder, F.Cu at (-48.1, 174.3)
- added D46: D_Small, Diode_SMD:D_0805_2012Metric_Pad1.15x1.40mm_HandSolder, F.Cu at (-48.1, 177.3)
- added D47: D_Small, Diode_SMD:D_0805_2012Metric_Pad1.15x1.40mm_HandSolder, F.Cu at (-48.1, 180.3)
- added D48: D_Small, Diode_SMD:D_0805_2012Metric_Pad1.15x1.40mm_HandSolder, F.Cu at (-48.1, 183.4)
- added D49: D_Small, Diode_SMD:D_0805_2012Metric_Pad1.15x1.40mm_HandSolder, F.Cu at (-48.1, 186.4)
- added D5: D_Small, Diode_SMD:D_0805_2012Metric_Pad1.15x1.40mm_HandSolder, F.Cu at (-62.5, 171.2)
- added D50: D_Small, Diode_SMD:D_0805_2012Metric_Pad1.15x1.40mm_HandSolder, F.Cu at (-48.1, 189.5)
- added D51: D_Small, Diode_SMD:D_0805_2012Metric_Pad1.15x1.40mm_HandSolder, F.Cu at (-48.1, 192.5)
- added D52: D_Small, Diode_SMD:D_0805_2012Metric_Pad1.15x1.40mm_HandSolder, F.Cu at (-48.1, 195.5)
- added D53: D_Small, Diode_SMD:D_0805_2012Metric_Pad1.15x1.40mm_HandSolder, F.Cu at (-43.3, 159.1)
- added D54: D_Small, Diode_SMD:D_0805_2012Metric_Pad1.15x1.40mm_HandSolder, F.Cu at (-43.3, 162.1)
- added D55: D_Small, Diode_SMD:D_0805_2012Metric_Pad1.15x1.40mm_HandSolder, F.Cu at (-43.3, 165.1)
- added D56: D_Small, Diode_SMD:D_0805_2012Metric_Pad1.15x1.40mm_HandSolder, F.Cu at (-43.3, 168.2)
- added D57: D_Small, Diode_SMD:D_0805_2012Metric_Pad1.15x1.40mm_HandSolder, F.Cu at (-43.3, 171.2)
- added D58: D_Small, Diode_SMD:D_0805_2012Metric_Pad1.15x1.40mm_HandSolder, F.Cu at (-43.3, 174.3)
- added D59: D_Small, Diode_SMD:D_0805_2012Metric_Pad1.15x1.40mm_HandSolder, F.Cu at (-43.3, 177.3)
- added D6: D_Small, Diode_SMD:D_0805_2012Metric_Pad1.15x1.40mm_HandSolder, F.Cu at (-62.5, 174.3)
- added D60: D_Small, Diode_SMD:D_0805_2012Metric_Pad1.15x1.40mm_HandSolder, F.Cu at (-43.3, 180.3)
- added D61: D_Small, Diode_SMD:D_0805_2012Metric_Pad1.15x1.40mm_HandSolder, F.Cu at (-43.3, 183.4)
- added D62: D_Small, Diode_SMD:D_0805_2012Metric_Pad1.15x1.40mm_HandSolder, F.Cu at (-43.3, 186.4)
- added D63: D_Small, Diode_SMD:D_0805_2012Metric_Pad1.15x1.40mm_HandSolder, F.Cu at (-43.3, 189.5)
- added D64: D_Small, Diode_SMD:D_0805_2012Metric_Pad1.15x1.40mm_HandSolder, F.Cu at (-43.3, 192.5)
- added D65: D_Small, Diode_SMD:D_0805_2012Metric_Pad1.15x1.40mm_HandSolder, F.Cu at (-43.3, 195.5)
- added D66: D_Small, Diode_SMD:D_0805_2012Metric_Pad1.15x1.40mm_HandSolder, F.Cu at (-38.5, 159.1)
- added D67: D_Small, Diode_SMD:D_0805_2012Metric_Pad1.15x1.40mm_HandSolder, F.Cu at (-38.5, 162.1)
- added D68: D_Small, Diode_SMD:D_0805_2012Metric_Pad1.15x1.40mm_HandSolder, F.Cu at (-38.5, 165.1)
- added D69: D_Small, Diode_SMD:D_0805_2012Metric_Pad1.15x1.40mm_HandSolder, F.Cu at (-38.5, 168.2)
- added D7: D_Small, Diode_SMD:D_0805_2012Metric_Pad1.15x1.40mm_HandSolder, F.Cu at (-62.5, 177.3)
- added D70: D_Small, Diode_SMD:D_0805_2012Metric_Pad1.15x1.40mm_HandSolder, F.Cu at (-38.5, 171.2)
- added D71: D_Small, Diode_SMD:D_0805_2012Metric_Pad1.15x1.40mm_HandSolder, F.Cu at (-38.5, 174.3)
- added D72: D_Small, Diode_SMD:D_0805_2012Metric_Pad1.15x1.40mm_HandSolder, F.Cu at (-38.5, 177.3)
- added D73: D_Small, Diode_SMD:D_0805_2012Metric_Pad1.15x1.40mm_HandSolder, F.Cu at (-38.5, 180.3)
- added D74: D_Small, Diode_SMD:D_0805_2012Metric_Pad1.15x1.40mm_HandSolder, F.Cu at (-38.5, 183.4)
- added D75: D_Small, Diode_SMD:D_0805_2012Metric_Pad1.15x1.40mm_HandSolder, F.Cu at (-38.5, 186.4)
- added D76: D_Small, Diode_SMD:D_0805_2012Metric_Pad1.15x1.40mm_HandSolder, F.Cu at (-38.5, 189.5)
- added D77: D_Small, Diode_SMD:D_0805_2012Metric_Pad1.15x1.40mm_HandSolder, F.Cu at (-38.5, 192.5)
- added D78: D_Small, Diode_SMD:D_0805_2012Metric_Pad1.15x1.40mm_HandSolder, F.Cu at (-38.5, 195.5)
- added D79: D_Small, Diode_SMD:D_0805_2012Metric_Pad1.15x1.40mm_HandSolder, F.Cu at (-33.7, 159.1)
- added D8: D_Small, Diode_SMD:D_0805_2012Metric_Pad1.15x1.40mm_HandSolder, F.Cu at (-62.5, 180.3)
- added D80: D_Small, Diode_SMD:D_0805_2012Metric_Pad1.15x1.40mm_HandSolder, F.Cu at (-33.7, 162.1)
- added D81: D_Small, Diode_SMD:D_0805_2012Metric_Pad1.15x1.40mm_HandSolder, F.Cu at (-33.7, 165.1)
- added D82: D_Small, Diode_SMD:D_0805_2012Metric_Pad1.15x1.40mm_HandSolder, F.Cu at (-33.7, 168.2)
- added D83: D_Small, Diode_SMD:D_0805_2012Metric_Pad1.15x1.40mm_HandSolder, F.Cu at (-33.7, 171.2)
- added D84: D_Small, Diode_SMD:D_0805_2012Metric_Pad1.15x1.40mm_HandSolder, F.Cu at (-33.7, 174.3)
- added D85: D_Small, Diode_SMD:D_0805_2012Metric_Pad1.15x1.40mm_HandSolder, F.Cu at (-33.7, 177.3)
- added D86: D_Small, Diode_SMD:D_0805_2012Metric_Pad1.15x1.40mm_HandSolder, F.Cu at (-33.7, 180.3)
- added D87: D_Small, Diode_SMD:D_0805_2012Metric_Pad1.15x1.40mm_HandSolder, F.Cu at (-33.7, 183.4)
- added D88: D_Small, Diode_SMD:D_0805_2012Metric_Pad1.15x1.40mm_HandSolder, F.Cu at (-33.7, 186.4)
- added D89: D_Small, Diode_SMD:D_0805_2012Metric_Pad1.15x1.40mm_HandSolder, F.Cu at (-33.7, 189.5)
- added D9: D_Small, Diode_SMD:D_0805_2012Metric_Pad1.15x1.40mm_HandSolder, F.Cu at (-62.5, 183.4)
- added D90: D_Small, Diode_SMD:D_0805_2012Metric_Pad1.15x1.40mm_HandSolder, F.Cu at (-33.7, 192.5)
- added D91: D_Small, Diode_SMD:D_0805_2012Metric_Pad1.15x1.40mm_HandSolder, F.Cu at (-33.7, 195.5)
- added D92: D_Small, Diode_SMD:D_0805_2012Metric_Pad1.15x1.40mm_HandSolder, F.Cu at (-28.9, 159.1)
- added D93: D_Small, Diode_SMD:D_0805_2012Metric_Pad1.15x1.40mm_HandSolder, F.Cu at (-28.9, 162.1)
- added D94: D_Small, Diode_SMD:D_0805_2012Metric_Pad1.15x1.40mm_HandSolder, F.Cu at (-28.9, 165.1)
- added D95: D_Small, Diode_SMD:D_0805_2012Metric_Pad1.15x1.40mm_HandSolder, F.Cu at (-28.9, 168.2)
- added D96: D_Small, Diode_SMD:D_0805_2012Metric_Pad1.15x1.40mm_HandSolder, F.Cu at (-28.9, 171.2)
- added D97: D_Small, Diode_SMD:D_0805_2012Metric_Pad1.15x1.40mm_HandSolder, F.Cu at (-28.9, 174.3)
- added D98: D_Small, Diode_SMD:D_0805_2012Metric_Pad1.15x1.40mm_HandSolder, F.Cu at (-28.9, 177.3)
- added D99: D_Small, Diode_SMD:D_0805_2012Metric_Pad1.15x1.40mm_HandSolder, F.Cu at (-28.9, 180.3)
- added F1: 500mA, Fuse:Fuse_1206_3216Metric_Pad1.42x1.75mm_HandSolder, F.Cu at (-112.2, 172.1)
- added J1: Conn_ARM_JTAG_SWD_10, Connector_PinSocket_2.54mm:PinSocket_2x05_P2.54mm_Vertical, F.Cu at (-122.1, 178.4)
- added R1: 22, Resistor_SMD:R_0805_2012Metric_Pad1.20x1.40mm_HandSolder, F.Cu at (-129.3, 177.6)
- added R2: 22, Resistor_SMD:R_0805_2012Metric_Pad1.20x1.40mm_HandSolder, F.Cu at (-129.3, 180.5)
- added R3: 5.1k, Resistor_SMD:R_0805_2012Metric_Pad1.20x1.40mm_HandSolder, F.Cu at (-129.3, 183.5)
- added R4: 5.1k, Resistor_SMD:R_0805_2012Metric_Pad1.20x1.40mm_HandSolder, F.Cu at (-129.3, 186.4)
- added R5: 10k, Resistor_SMD:R_0805_2012Metric_Pad1.20x1.40mm_HandSolder, F.Cu at (-129.3, 189.4)
- added R6: 10k, Resistor_SMD:R_0805_2012Metric_Pad1.20x1.40mm_HandSolder, F.Cu at (-129.3, 192.3)
- added SW1: ESC, Kailh_PG1353_Hotswap:Kailh-PG1353-Hotswap-1.5U, F.Cu at (54.8, 34.6)
- added SW10: F9, Kailh_PG1353_Hotswap:Kailh-PG1353-Hotswap-1U, F.Cu at (230.9, 34.6)
- added SW100: SW_Push_Dual, random-keyboard-parts.pretty-master:SKQG-1155865, F.Cu at (-115.0, 189.9)
- added SW11: F10, Kailh_PG1353_Hotswap:Kailh-PG1353-Hotswap-1U, F.Cu at (250.0, 34.6)
- added SW12: F11, Kailh_PG1353_Hotswap:Kailh-PG1353-Hotswap-1U, F.Cu at (269.1, 34.6)
- added SW13: F12, Kailh_PG1353_Hotswap:Kailh-PG1353-Hotswap-1U, F.Cu at (288.1, 34.6)
- added SW14: PWR, Kailh_PG1353_Hotswap:Kailh-PG1353-Hotswap-1.5U, F.Cu at (311.9, 34.6)
- added SW15: NUMLCK, Kailh_PG1353_Hotswap:Kailh-PG1353-Hotswap-1U, F.Cu at (415.6, 41.6)
- added SW16: DIV, Kailh_PG1353_Hotswap:Kailh-PG1353-Hotswap-1U, F.Cu at (438.6, 41.1)
- added SW17: MULT, Kailh_PG1353_Hotswap:Kailh-PG1353-Hotswap-1U, F.Cu at (462.1, 42.6)
- added SW18: SUB, Kailh_PG1353_Hotswap:Kailh-PG1353-Hotswap-1U, F.Cu at (485.1, 42.6)
- added SW19: /, Kailh_PG1353_Hotswap:Kailh-PG1353-Hotswap-1U, F.Cu at (50.0, 53.6)
- added SW2: F1, Kailh_PG1353_Hotswap:Kailh-PG1353-Hotswap-1U, F.Cu at (78.6, 34.6)
- added SW20: 1, Kailh_PG1353_Hotswap:Kailh-PG1353-Hotswap-1U, F.Cu at (69.0, 53.6)
- added SW21: 2, Kailh_PG1353_Hotswap:Kailh-PG1353-Hotswap-1U, F.Cu at (88.1, 53.6)
- added SW22: 3, Kailh_PG1353_Hotswap:Kailh-PG1353-Hotswap-1U, F.Cu at (107.2, 53.6)
- added SW23: 4, Kailh_PG1353_Hotswap:Kailh-PG1353-Hotswap-1U, F.Cu at (126.2, 53.6)
- added SW24: 5, Kailh_PG1353_Hotswap:Kailh-PG1353-Hotswap-1U, F.Cu at (145.3, 53.6)
- added SW25: 6, Kailh_PG1353_Hotswap:Kailh-PG1353-Hotswap-1U, F.Cu at (164.3, 53.6)
- added SW26: 7, Kailh_PG1353_Hotswap:Kailh-PG1353-Hotswap-1U, F.Cu at (183.4, 53.6)
- added SW27: 8, Kailh_PG1353_Hotswap:Kailh-PG1353-Hotswap-1U, F.Cu at (202.4, 53.6)
- added SW28: 9, Kailh_PG1353_Hotswap:Kailh-PG1353-Hotswap-1U, F.Cu at (221.4, 53.6)
- added SW29: 0, Kailh_PG1353_Hotswap:Kailh-PG1353-Hotswap-1U, F.Cu at (240.5, 53.6)
- added SW3: F2, Kailh_PG1353_Hotswap:Kailh-PG1353-Hotswap-1U, F.Cu at (97.6, 34.6)
- added SW30: -, Kailh_PG1353_Hotswap:Kailh-PG1353-Hotswap-1U, F.Cu at (259.6, 53.6)
- added SW31: =, Kailh_PG1353_Hotswap:Kailh-PG1353-Hotswap-1U, F.Cu at (278.6, 53.6)
- added SW32: DEL, Kailh_PG1353_Hotswap:Kailh-PG1353-Hotswap-2U, F.Cu at (307.2, 53.6)
- added SW33: #7, Kailh_PG1353_Hotswap:Kailh-PG1353-Hotswap-1U, F.Cu at (415.0, 62.5)
- added SW34: #8, Kailh_PG1353_Hotswap:Kailh-PG1353-Hotswap-1U, F.Cu at (438.1, 62.6)
- added SW35: #9, Kailh_PG1353_Hotswap:Kailh-PG1353-Hotswap-1U, F.Cu at (461.5, 64.0)
- added SW36: TAB, Kailh_PG1353_Hotswap:Kailh-PG1353-Hotswap-1.5U, F.Cu at (54.8, 72.7)
- added SW37: Q, Kailh_PG1353_Hotswap:Kailh-PG1353-Hotswap-1U, F.Cu at (78.5, 72.7)
- added SW38: W, Kailh_PG1353_Hotswap:Kailh-PG1353-Hotswap-1U, F.Cu at (97.6, 72.7)
- added SW39: E, Kailh_PG1353_Hotswap:Kailh-PG1353-Hotswap-1U, F.Cu at (116.7, 72.7)
- added SW4: F3, Kailh_PG1353_Hotswap:Kailh-PG1353-Hotswap-1U, F.Cu at (116.7, 34.6)
- added SW40: R, Kailh_PG1353_Hotswap:Kailh-PG1353-Hotswap-1U, F.Cu at (135.7, 72.7)
- added SW41: T, Kailh_PG1353_Hotswap:Kailh-PG1353-Hotswap-1U, F.Cu at (154.8, 72.7)
- added SW42: Y, Kailh_PG1353_Hotswap:Kailh-PG1353-Hotswap-1U, F.Cu at (173.8, 72.7)
- added SW43: U, Kailh_PG1353_Hotswap:Kailh-PG1353-Hotswap-1U, F.Cu at (192.9, 72.7)
- added SW44: I, Kailh_PG1353_Hotswap:Kailh-PG1353-Hotswap-1U, F.Cu at (211.9, 72.7)
- added SW45: O, Kailh_PG1353_Hotswap:Kailh-PG1353-Hotswap-1U, F.Cu at (231.0, 72.7)
- added SW46: P, Kailh_PG1353_Hotswap:Kailh-PG1353-Hotswap-1U, F.Cu at (250.0, 72.7)
- added SW47: ^, Kailh_PG1353_Hotswap:Kailh-PG1353-Hotswap-1U, F.Cu at (269.1, 72.7)
- added SW48: Ç, Kailh_PG1353_Hotswap:Kailh-PG1353-Hotswap-1U, F.Cu at (288.1, 72.7)
- added SW49: ENTER, Kailh_PG1353_Hotswap:Kailh-PG1353-Hotswap-1.5U, F.Cu at (311.9, 72.7)
- added SW5: F4, Kailh_PG1353_Hotswap:Kailh-PG1353-Hotswap-1U, F.Cu at (135.7, 34.6)
- added SW50: #4, Kailh_PG1353_Hotswap:Kailh-PG1353-Hotswap-1U, F.Cu at (415.0, 85.5)
- added SW51: #5, Kailh_PG1353_Hotswap:Kailh-PG1353-Hotswap-1U, F.Cu at (438.1, 85.6)
- added SW52: #6, Kailh_PG1353_Hotswap:Kailh-PG1353-Hotswap-1U, F.Cu at (462.1, 86.1)
- added SW53: ADD, Kailh_PG1353_Hotswap:Kailh-PG1353-Hotswap-2U, F.Cu at (485.5, 75.0)
- added SW54: CAPSLCK, Kailh_PG1353_Hotswap:Kailh-PG1353-Hotswap-1.75U, F.Cu at (57.1, 91.8)
- added SW55: A, Kailh_PG1353_Hotswap:Kailh-PG1353-Hotswap-1U, F.Cu at (83.3, 91.8)
- added SW56: S, Kailh_PG1353_Hotswap:Kailh-PG1353-Hotswap-1U, F.Cu at (102.4, 91.8)
- added SW57: D, Kailh_PG1353_Hotswap:Kailh-PG1353-Hotswap-1U, F.Cu at (121.5, 91.8)
- added SW58: F, Kailh_PG1353_Hotswap:Kailh-PG1353-Hotswap-1U, F.Cu at (140.5, 91.8)
- added SW59: G, Kailh_PG1353_Hotswap:Kailh-PG1353-Hotswap-1U, F.Cu at (159.6, 91.8)
- added SW6: F5, Kailh_PG1353_Hotswap:Kailh-PG1353-Hotswap-1U, F.Cu at (154.8, 34.6)
- added SW60: H, Kailh_PG1353_Hotswap:Kailh-PG1353-Hotswap-1U, F.Cu at (178.6, 91.8)
- added SW61: J, Kailh_PG1353_Hotswap:Kailh-PG1353-Hotswap-1U, F.Cu at (197.7, 91.8)
- added SW62: K, Kailh_PG1353_Hotswap:Kailh-PG1353-Hotswap-1U, F.Cu at (216.7, 91.8)
- added SW63: L, Kailh_PG1353_Hotswap:Kailh-PG1353-Hotswap-1U, F.Cu at (235.8, 91.8)
- added SW64: ;, Kailh_PG1353_Hotswap:Kailh-PG1353-Hotswap-1U, F.Cu at (254.8, 91.8)
- added SW65: È, Kailh_PG1353_Hotswap:Kailh-PG1353-Hotswap-1U, F.Cu at (273.9, 91.8)
- added SW66: À, Kailh_PG1353_Hotswap:Kailh-PG1353-Hotswap-1U, F.Cu at (292.9, 91.8)
- added SW67: ENTER, Kailh_PG1353_Hotswap:Kailh-PG1353-Hotswap-1.25U, F.Cu at (314.4, 91.8)
- added SW68: #1, Kailh_PG1353_Hotswap:Kailh-PG1353-Hotswap-1U, F.Cu at (416.1, 108.1)
- added SW69: #2, Kailh_PG1353_Hotswap:Kailh-PG1353-Hotswap-1U, F.Cu at (441.5, 109.0)
- added SW7: F6, Kailh_PG1353_Hotswap:Kailh-PG1353-Hotswap-1U, F.Cu at (173.8, 34.6)
- added SW70: #3, Kailh_PG1353_Hotswap:Kailh-PG1353-Hotswap-1U, F.Cu at (465.1, 109.1)
- added SW71: #ENTER, Kailh_PG1353_Hotswap:Kailh-PG1353-Hotswap-2U, F.Cu at (487.6, 117.4)
- added SW72: LSHFT, Kailh_PG1353_Hotswap:Kailh-PG1353-Hotswap-1.25U, F.Cu at (52.4, 110.8)
- added SW73: Ù, Kailh_PG1353_Hotswap:Kailh-PG1353-Hotswap-1U, F.Cu at (73.8, 110.8)
- added SW74: Z, Kailh_PG1353_Hotswap:Kailh-PG1353-Hotswap-1U, F.Cu at (92.9, 110.8)
- added SW75: X, Kailh_PG1353_Hotswap:Kailh-PG1353-Hotswap-1U, F.Cu at (111.9, 110.8)
- added SW76: C, Kailh_PG1353_Hotswap:Kailh-PG1353-Hotswap-1U, F.Cu at (131.0, 110.8)
- added SW77: V, Kailh_PG1353_Hotswap:Kailh-PG1353-Hotswap-1U, F.Cu at (150.0, 110.8)
- added SW78: B, Kailh_PG1353_Hotswap:Kailh-PG1353-Hotswap-1U, F.Cu at (169.1, 110.8)
- added SW79: N, Kailh_PG1353_Hotswap:Kailh-PG1353-Hotswap-1U, F.Cu at (188.1, 110.8)
- added SW8: F7, Kailh_PG1353_Hotswap:Kailh-PG1353-Hotswap-1U, F.Cu at (192.9, 34.6)
- added SW80: M, Kailh_PG1353_Hotswap:Kailh-PG1353-Hotswap-1U, F.Cu at (207.2, 110.8)
- added SW81: ,, Kailh_PG1353_Hotswap:Kailh-PG1353-Hotswap-1U, F.Cu at (226.2, 110.8)
- added SW82: ., Kailh_PG1353_Hotswap:Kailh-PG1353-Hotswap-1U, F.Cu at (245.3, 110.8)
- added SW83: É, Kailh_PG1353_Hotswap:Kailh-PG1353-Hotswap-1U, F.Cu at (264.3, 110.8)
- added SW84: RSHFT, Kailh_PG1353_Hotswap:Kailh-PG1353-Hotswap-2.75U, F.Cu at (300.0, 110.8)
- added SW85: INSERT, Kailh_PG1353_Hotswap:Kailh-PG1353-Hotswap-2U, F.Cu at (425.6, 130.6)
- added SW86: UP ARROW, Kailh_PG1353_Hotswap:Kailh-PG1353-Hotswap-1U, F.Cu at (463.1, 131.6)
- added SW87: FN, Kailh_PG1353_Hotswap:Kailh-PG1353-Hotswap-1U, F.Cu at (50.0, 129.8)
- added SW88: CRTL, Kailh_PG1353_Hotswap:Kailh-PG1353-Hotswap-1U, F.Cu at (69.0, 129.8)
- added SW89: LOPT, Kailh_PG1353_Hotswap:Kailh-PG1353-Hotswap-1U, F.Cu at (88.1, 129.8)
- added SW9: F8, Kailh_PG1353_Hotswap:Kailh-PG1353-Hotswap-1U, F.Cu at (211.9, 34.6)
- added SW90: LCMD, Kailh_PG1353_Hotswap:Kailh-PG1353-Hotswap-1.25U, F.Cu at (109.5, 129.8)
- added SW91: SPACE, Kailh_PG1353_Hotswap:Kailh-PG1353-Hotswap-6.25U, F.Cu at (181.0, 129.8)
- added SW92: RCMD, Kailh_PG1353_Hotswap:Kailh-PG1353-Hotswap-1.25U, F.Cu at (252.4, 129.8)
- added SW93: ROPT, Kailh_PG1353_Hotswap:Kailh-PG1353-Hotswap-1U, F.Cu at (273.8, 129.8)
- added SW94: B0, Kailh_PG1353_Hotswap:Kailh-PG1353-Hotswap-1.25U, F.Cu at (295.3, 129.8)
- added SW95: B1, Kailh_PG1353_Hotswap:Kailh-PG1353-Hotswap-1U, F.Cu at (316.7, 129.8)
- added SW96: #DEL, Kailh_PG1353_Hotswap:Kailh-PG1353-Hotswap-1U, F.Cu at (415.5, 155.5)
- added SW97: LEFT ARROW, Kailh_PG1353_Hotswap:Kailh-PG1353-Hotswap-1U, F.Cu at (438.1, 154.6)
- added SW98: DOWN ARROW, Kailh_PG1353_Hotswap:Kailh-PG1353-Hotswap-1U, F.Cu at (463.0, 157.5)
- added SW99: RIGHT ARROW, Kailh_PG1353_Hotswap:Kailh-PG1353-Hotswap-1U, F.Cu at (487.6, 155.6)
- added U1: PRTR5V0U2X, random-keyboard-parts.pretty-master:SOT143B, F.Cu at (-111.7, 166.8)
- added U2: STM32F072CBTx, Package_QFP:LQFP-48_7x7mm_P0.5mm, F.Cu at (-126.0, 170.4)
- added U3: AP2112K-3.3, Package_TO_SOT_SMD:SOT-23-5, F.Cu at (-117.8, 172.9)
- added USB1: HRO-TYPE-C-31-M-12, Type-C.pretty-master:HRO-TYPE-C-31-M-12-HandSoldering, F.Cu at (-114.5, 186.0)
- added Y1: 8MHz, Crystal:Crystal_SMD_3225-4Pin_3.2x2.5mm_HandSoldering, F.Cu at (-117.0, 167.6)

Commit message: numpad diodes placed
Parts:
- D15, D16, D17, D18, D33, D34, D35, D50, D51, D52, D53, D68, D69, D70, D71, D85, D86, D96, D97, D98, D99: moved to B.Cu
- moved D18 490.1 mm to (413.0, 34.5), turned to 90 degrees
- moved D17 471.0 mm to (394.0, 34.5), turned to 90 degrees
- moved D35 465.4 mm to (394.0, 53.5), turned to 90 degrees
- moved D53 461.4 mm to (406.6, 56.6), turned to 180 degrees
- moved D52 458.9 mm to (394.0, 72.5), turned to 90 degrees
- moved D71 452.5 mm to (407.0, 95.0), turned to 180 degrees
- moved D16 451.9 mm to (375.0, 34.5), turned to 90 degrees
- moved D34 446.3 mm to (375.0, 53.5), turned to 90 degrees
- moved D99 444.8 mm to (413.0, 129.5), turned to 90 degrees
- moved D70 439.8 mm to (394.0, 91.5), turned to 90 degrees
- moved D51 439.8 mm to (375.0, 72.5), turned to 90 degrees
- moved D86 433.3 mm to (394.0, 110.5), turned to 90 degrees
- moved D15 432.9 mm to (356.0, 34.5), turned to 90 degrees
- moved D33 427.2 mm to (356.0, 53.5), turned to 90 degrees
- moved D98 425.6 mm to (394.0, 129.5), turned to 90 degrees
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
Commit message: all diodes placed
Parts:
- D1, D10, D11, D12, D13, D14, D19, D2, D20, D21, D22, D23, D24, D25, D26, D27, D28, D29, D3, D30, D31, D32, D36, D37, D38, D39, D4, D40, D41, D42, D43, D44, D45, D46, D47, D48, D49, D5, D54, D55, D56, D57, D58, D59, D6, D60, D61, D62, D63, D64, D65, D66, D67, D7, D72, D73, D74, D75, D76, D77, D78, D79, D8, D80, D81, D82, D83, D84, D87, D88, D89, D9, D90, D91, D92, D93, D94, D95: moved to B.Cu
- moved U2 149.0 mm to (202.9, 162.6)
- moved D72 28.2 mm to (33.3, 105.1), turned to 90 degrees
- moved D36 27.5 mm to (35.8, 67.0), turned to 90 degrees
- moved D42 27.4 mm to (154.3, 67.0), turned to 90 degrees
- moved D14 27.4 mm to (292.8, 29.1), turned to 90 degrees
- moved D21 27.2 mm to (68.8, 48.0), turned to 90 degrees
- moved D32 27.1 mm to (288.3, 48.0), turned to 90 degrees
- moved D44 27.1 mm to (192.8, 67.0), turned to 90 degrees
- moved D54 27.1 mm to (37.8, 86.1), turned to 90 degrees
- moved D6 27.1 mm to (135.8, 29.0), turned to 90 degrees
- moved D48 26.9 mm to (268.8, 67.0), turned to 90 degrees
- moved D77 26.9 mm to (130.8, 105.0), turned to 90 degrees
- moved D46 26.9 mm to (230.8, 67.0), turned to 90 degrees
- moved D37 26.9 mm to (59.3, 67.1), turned to 90 degrees
- moved D45 26.8 mm to (211.8, 67.1), turned to 90 degrees
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
Commit message: other components placed + contours
Parts:
- C1, C2, C3, C4, C5, C6, C7, C8, C9, F1, J1, R1, R2, R3, R4, R5, R6, SW100, U1, U2, U3, USB1, Y1: moved to B.Cu
- moved USB1 182.3 mm to (157.8, 24.8)
- moved R3 181.0 mm to (158.5, 37.0)
- moved R4 179.2 mm to (152.5, 37.0), turned to 180 degrees
- moved F1 152.8 mm to (156.5, 46.5), turned to -90 degrees
- moved U1 152.5 mm to (161.5, 46.0), turned to 180 degrees
- moved SW100 137.8 mm to (181.5, 139.5), turned to 90 degrees
- moved J1 132.4 mm to (170.0, 132.3), turned to 180 degrees
- moved C9 120.4 mm to (145.5, 144.0), turned to 180 degrees
- moved C7 119.8 mm to (145.5, 140.5), turned to 180 degrees
- moved C8 111.6 mm to (136.5, 141.5), turned to 180 degrees
- moved R5 109.1 mm to (136.5, 137.0), turned to 180 degrees
- moved C5 105.4 mm to (133.0, 144.5), turned to 90 degrees
- moved R2 102.7 mm to (130.0, 129.0), turned to -90 degrees
- moved R6 99.7 mm to (128.5, 145.5), turned to 180 degrees
- moved R1 99.3 mm to (127.5, 129.0), turned to -90 degrees
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Other:
- board outline added: 392 x 122 mm

Commit message: midway correcting hotswap sockets
Parts:
- added J2: Conn_01x04_Socket, pogo_conn_4_pins:686L0421350120E, B.Cu at (299.5, 54.1)
- added J3: Conn_01x04_Pin, pogo_conn_4_pins:685L0421250110E, B.Cu at (328.8, 54.2)
- added J4: Conn_01x03_Socket, pogo_conn_3_pins:685F0321351124E, B.Cu at (299.6, 88.0)
- added J5: Conn_01x03_Pin, pogo_conn_3_pins:685F0321350124E, B.Cu at (328.9, 84.0)
- added J6: Conn_01x03_Socket, pogo_conn_3_pins:685F0321351124E, B.Cu at (299.6, 120.2)
- added J7: Conn_01x03_Pin, pogo_conn_3_pins:685F0321350124E, B.Cu at (328.9, 116.2)
- D19, D20, D21, D22, D23, D24, D25, D26, D27, D28, D29, D30, D31, D32, D36, D49, D54, D67, D72, D84, D87, D95: moved to F.Cu
- SW1, SW10, SW11, SW12, SW13, SW14, SW19, SW2, SW20, SW21, SW22, SW23, SW24, SW25, SW26, SW27, SW28, SW29, SW3, SW30, SW31, SW32, SW36, SW4, SW49, SW5, SW54, SW6, SW67, SW7, SW72, SW8, SW84, SW87, SW9, SW95: moved to B.Cu
- moved R6 15.2 mm to (118.5, 134.0), turned to 0 degrees
- moved C6 15.2 mm to (119.8, 130.8), turned to -90 degrees
- moved C3 14.8 mm to (117.2, 130.8), turned to 90 degrees
- moved D22 13.7 mm to (74.6, 61.0)
- moved D32 13.6 mm to (274.6, 61.0)
- moved D84 13.6 mm to (267.5, 118.0)
- moved D95 13.6 mm to (284.2, 137.1)
- moved D5 13.6 mm to (103.2, 42.1)
- moved D23 13.6 mm to (93.7, 61.0)
- moved D1 13.5 mm to (22.3, 42.0)
- moved D36 13.5 mm to (22.3, 80.0)
- moved D6 13.5 mm to (122.3, 42.0)
- moved D24 13.5 mm to (112.8, 61.0)
- moved D25 13.4 mm to (131.9, 61.0)
- moved D67 13.3 mm to (282.0, 99.0)
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Connections:
- D15 pad 1: ROW0B -> ROW0C
- D16 pad 1: ROW0B -> ROW0C
- D17 pad 1: ROW0B -> ROW0C
- D18 pad 1: ROW0B -> ROW0C
- D33 pad 1: ROW1B -> ROW1C
- D34 pad 1: ROW1B -> ROW1C
- D35 pad 1: ROW1B -> ROW1C
- D50 pad 1: ROW2B -> ROW2C
- D51 pad 1: ROW2B -> ROW2C
- D52 pad 1: ROW2B -> ROW2C
- D53 pad 1: ROW2B -> ROW2C
- D68 pad 1: ROW3B -> ROW3C
- D69 pad 1: ROW3B -> ROW3C
- D70 pad 1: ROW3B -> ROW3C
- D71 pad 1: ROW3B -> ROW3C
- D85 pad 1: ROW4B -> ROW4C
- D86 pad 1: ROW4B -> ROW4C
- D91 pad 1: ROW5A -> ROW5B
- D96 pad 1: ROW5B -> ROW5C
- D97 pad 1: ROW5B -> ROW5C
- D98 pad 1: ROW5B -> ROW5C
- D99 pad 1: ROW5B -> ROW5C
- U2 pad 10: COL0 -> unconnected-(U2-PA0-Pad10)
- U2 pad 11: COL1 -> unconnected-(U2-PA1-Pad11)
- U2 pad 12: COL2 -> COL0
- U2 pad 13: COL3 -> COL1
- U2 pad 14: COL4 -> COL2
- U2 pad 15: COL5 -> COL3
- U2 pad 16: COL6 -> COL4
- U2 pad 17: COL14 -> COL5
- U2 pad 18: ROW0A -> COL6
- U2 pad 19: ROW1A -> ROW0A
- U2 pad 20: ROW2A -> ROW0B
- U2 pad 21: ROW4B -> ROW1B
- U2 pad 22: ROW5B -> unconnected-(U2-PB11-Pad22)
- U2 pad 25: unconnected-(U2-PB12-Pad25) -> SWCLK
- U2 pad 26: unconnected-(U2-PB13-Pad26) -> SWDIO
- U2 pad 28: unconnected-(U2-PB15-Pad28) -> ROW2B
- U2 pad 29: COL15 -> ROW3B
- U2 pad 30: COL16 -> ROW4B
- U2 pad 31: COL17 -> ROW5B
- U2 pad 34: SWDIO -> unconnected-(U2-PA13-Pad34)
- U2 pad 37: SWCLK -> Net-(J2-Pin_4)
- U2 pad 38: unconnected-(U2-PA15-Pad38) -> Net-(J2-Pin_3)
- U2 pad 39: ROW3A -> Net-(J2-Pin_2)
- U2 pad 40: ROW4A -> Net-(J2-Pin_1)
- U2 pad 42: ROW0B -> ROW4A
- U2 pad 43: ROW1B -> ROW3A
- U2 pad 45: ROW2B -> ROW2A
- U2 pad 46: ROW3B -> ROW1A
Routing:
- net COL0: track 0.00 -> 312.2 mm, vias 0 -> 1
- net Net-(J2-Pin_1): track 0.00 -> 294.0 mm, vias 0 -> 5
- net Net-(J2-Pin_2): track 0.00 -> 292.8 mm, vias 0 -> 5
- net Net-(J2-Pin_3): track 0.00 -> 292.2 mm, vias 0 -> 5
- net Net-(J2-Pin_4): track 0.00 -> 292.1 mm, vias 0 -> 5
- net COL1: track 0.00 -> 274.4 mm, vias 0 -> 3
- net COL2: track 0.00 -> 235.8 mm, vias 0 -> 3
- net COL3: track 0.00 -> 192.9 mm, vias 0 -> 3
- net GND: track 0.00 -> 190.8 mm, vias 0 -> 3
- net COL17: track 0.00 -> 165.9 mm, vias 0 -> 3
- net COL4: track 0.00 -> 144.8 mm, vias 0 -> 3
- net COL5: track 0.00 -> 142.0 mm, vias 0 -> 3
- net COL16: track 0.00 -> 135.0 mm, vias 0 -> 3
- net COL15: track 0.00 -> 123.6 mm, vias 0 -> 1
- net ROW0C: track 0.00 -> 112.0 mm
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- added copper zone on B.Cu, net GND
Other:
- board size 392 x 122 mm -> 392 x 125.2 mm

Commit message: 1/3 of matrix re-routed
Parts:
- D19, D20, D21, D22, D23, D24, D25, D26, D27, D28, D29, D30, D31, D32, D36, D49, D54, D67, D72, D84, D87, D95, SW15, SW16, SW17, SW18, SW33, SW34, SW35, SW37, SW38, SW39, SW40, SW41, SW42, SW43, SW44, SW45, SW46, SW47, SW48, SW50, SW51, SW52, SW53, SW55, SW56, SW57, SW58, SW59, SW60, SW61, SW62, SW63, SW64, SW65, SW66, SW68, SW69, SW70, SW71, SW73, SW74, SW75, SW76, SW77, SW78, SW79, SW80, SW81, SW82, SW83, SW85, SW86, SW88, SW89, SW90, SW91, SW92, SW93, SW94, SW96, SW97, SW98, SW99: moved to B.Cu
- moved D38 13.8 mm to (65.0, 80.0)
- moved D39 13.7 mm to (84.1, 80.0)
- moved D40 13.6 mm to (103.2, 80.0)
- moved D63 13.5 mm to (203.2, 99.1)
- moved D41 13.5 mm to (122.3, 80.0)
- moved D94 13.4 mm to (262.8, 137.1)
- moved D64 13.4 mm to (222.3, 99.1)
- moved D55 13.4 mm to (50.9, 99.1)
- moved D73 13.4 mm to (41.4, 118.0)
- moved D65 13.3 mm to (241.4, 99.1)
- moved D93 13.3 mm to (241.5, 137.1)
- moved D43 13.3 mm to (160.5, 80.1)
- moved D75 13.2 mm to (79.6, 118.1)
- moved D56 13.2 mm to (70.1, 99.0)
- moved D66 13.2 mm to (260.6, 99.0)
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Routing:
- net COL17: track 165.9 -> 0.00 mm, vias 3 -> 0
- net COL2: track 235.8 -> 398.4 mm, vias 3 -> 15
- net COL1: track 274.4 -> 433.6 mm, vias 3 -> 15
- net COL5: track 142.0 -> 297.9 mm, vias 3 -> 13
- net COL3: track 192.9 -> 340.0 mm, vias 3 -> 15
- net COL4: track 144.8 -> 289.6 mm, vias 3 -> 13
- net COL0: track 312.2 -> 453.4 mm, vias 1 -> 12
- net COL16: track 135.0 -> 0.00 mm, vias 3 -> 0
- net ROW0A: track 10.3 -> 142.6 mm
- net ROW3A: track 59.0 -> 190.8 mm
- net ROW2A: track 55.8 -> 185.5 mm
- net ROW1A: track 53.1 -> 177.7 mm
- net COL15: track 123.6 -> 0.00 mm, vias 1 -> 0
- net ROW4A: track 58.0 -> 173.2 mm
- net ROW0C: track 112.0 -> 0.00 mm
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
Commit message: new connectors placed
Parts:
- removed J6: Conn_01x03_Socket, pogo_conn_3_pins:685F0321351124E
- removed J7: Conn_01x03_Pin, pogo_conn_3_pins:685F0321350124E
- added FB1: FerriteBead_Small, Inductor_SMD:L_0805_2012Metric_Pad1.05x1.20mm_HandSolder, B.Cu at (151.5, 33.4)
- J2: value Conn_01x04_Socket -> Conn_01x05_Socket; footprint pogo_conn_4_pins:686L0421350120E -> pogo_connector_5_pins:female; moved to F.Cu
- J3: value Conn_01x04_Pin -> Conn_01x05_Pin; footprint pogo_conn_4_pins:685L0421250110E -> pogo_connector_5_pins:male; moved to F.Cu
- J4: value Conn_01x03_Socket -> Conn_01x05_Socket; footprint pogo_conn_3_pins:685F0321351124E -> pogo_connector_5_pins:female; moved to F.Cu
- J5: value Conn_01x03_Pin -> Conn_01x05_Pin; footprint pogo_conn_3_pins:685F0321350124E -> pogo_connector_5_pins:male; moved to F.Cu
- moved J2 68.3 mm to (299.5, 122.4), turned to 180 degrees
- moved J3 68.2 mm to (329.0, 122.4), turned to 180 degrees
- moved J4 34.4 mm to (299.5, 49.8), turned to 180 degrees
- moved J5 30.4 mm to (329.0, 49.8), turned to 180 degrees
Connections:
- J2 pad 1: Net-(J2-Pin_1) -> ROW5B
- J2 pad 2: Net-(J2-Pin_2) -> ROW4B
- J2 pad 3: Net-(J2-Pin_3) -> ROW3B
- J2 pad 4: Net-(J2-Pin_4) -> ROW2B
- J3 pad 1: COL17 -> ROW1C
- J3 pad 2: COL16 -> ROW2C
- J3 pad 3: COL15 -> ROW3C
- J3 pad 4: COL14 -> ROW4C
- J4 pad 1: ROW2B -> COL17MAIN
- J4 pad 2: ROW1B -> COL16MAIN
- J4 pad 3: ROW0B -> COL15MAIN
- J5 pad 1: ROW2C -> ROW0C
- J5 pad 2: ROW1C -> COL17
- J5 pad 3: ROW0C -> COL16
- U2 pad 37: Net-(J2-Pin_4) -> COL14MAIN
- U2 pad 38: Net-(J2-Pin_3) -> COL15MAIN
- U2 pad 39: Net-(J2-Pin_2) -> COL16MAIN
- U2 pad 40: Net-(J2-Pin_1) -> COL17MAIN
- USB1 pad 13: GND -> Earth
Routing:
- net Net-(J2-Pin_1): track 294.2 -> 0.00 mm, vias 5 -> 0
- net Net-(J2-Pin_2): track 293.0 -> 0.00 mm, vias 5 -> 0
- net Net-(J2-Pin_3): track 292.4 -> 0.00 mm, vias 5 -> 0
- net Net-(J2-Pin_4): track 292.3 -> 0.00 mm, vias 5 -> 0
- net COL17MAIN: track 0.00 -> 273.8 mm, vias 0 -> 5
- net COL15MAIN: track 0.00 -> 273.6 mm, vias 0 -> 5
- net COL16MAIN: track 0.00 -> 273.6 mm, vias 0 -> 5
- net COL14MAIN: track 0.00 -> 273.1 mm, vias 0 -> 5
- net COL17: track 0.00 -> 199.5 mm, vias 0 -> 6
- net COL16: track 0.00 -> 176.0 mm, vias 0 -> 8
- net COL15: track 0.00 -> 153.1 mm, vias 0 -> 7
- net COL14: track 0.00 -> 147.7 mm, vias 0 -> 6
- net ROW1B: track 14.8 -> 151.7 mm
- net ROW2B: track 24.6 -> 157.0 mm
- net ROW3B: track 36.4 -> 166.0 mm
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Other:
- board size 392 x 125.2 mm -> 392.5 x 125.2 mm
