File: new-keyboard-pcb/new-keyboard-pcb.kicad_pcb (KiCad board)
At the start: 2 copper layers, 392.5 x 125.2 mm, 226 parts, among them J1 Conn_ARM_JTAG_SWD_10, J2 Conn_01x05_Socket, J3 Conn_01x05_Pin, J4 Conn_01x05_Socket, J5 Conn_01x05_Pin, SW1 ESC, SW10 F9, SW100 SW_Push_Dual, SW11 F10, SW12 F11, SW13 F12, SW14 PWR, SW15 NUMLCK, SW16 DIV, SW17 MULT, SW18 SUB, SW19 /, SW2 F1, SW20 1, SW21 2, SW22 3, SW23 4, SW24 5, SW25 6, SW26 7, SW27 8, SW28 9, SW29 0, SW3 F2, SW30 -, SW31 =, SW32 DEL, SW33 #7, SW34 #8, SW35 #9, SW36 TAB, SW37 Q, SW38 W, SW39 E, SW4 F3, SW40 R, SW41 T, SW42 Y, SW43 U, SW44 I, SW45 O, SW46 P, SW47 ^, SW48 Ç, SW49 ENTER, SW5 F4, SW50 #4, SW51 #5, SW52 #6, SW53 ADD, SW54 CAPSLCK, SW55 A, SW56 S, SW57 D, SW58 F, SW59 G, SW6 F5, SW60 H, SW61 J, SW62 K, SW63 L, SW64 ;, SW65 È, SW66 À, SW67 ENTER, SW68 #1, SW69 #2, SW7 F6, SW70 #3, SW71 #ENTER, SW72 LSHFT, SW73 Ù, SW74 Z, SW75 X, SW76 C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

Commit message: everything routed (again)
Parts:
- moved D91 2.55 mm to (148.7, 134.5)
Routing:
- net COL6: track 83.5 -> 311.6 mm
- net ROW1B: track 151.7 -> 295.5 mm, vias 3 -> 6
- net COL3: track 340.0 -> 471.1 mm
- net COL2: track 398.4 -> 529.0 mm
- net COL1: track 433.6 -> 561.1 mm
- net ROW0B: track 144.3 -> 270.8 mm, vias 3 -> 8
- net COL4: track 289.6 -> 412.8 mm
- net COL0: track 453.4 -> 573.0 mm
- net GND: track 149.9 -> 269.5 mm, vias 1 -> 7
- net COL5: track 297.9 -> 404.1 mm
- net ROW2B: track 157.0 -> 258.1 mm, vias 0 -> 2
- net +5V: track 49.7 -> 136.6 mm, vias 2 -> 4
- net Net-(U1-IO1): track 50.7 -> 134.4 mm, vias 0 -> 2
- net Net-(U1-IO2): track 50.4 -> 133.4 mm, vias 0 -> 2
- net ROW0A: track 142.6 -> 224.1 mm, vias 3 -> 4
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